File: sensor-breakout-boards/emstat-to-usb-sensor.brd (EAGLE design)
At the start: 24 x 30 mm, 4 parts, among them X1 Type-A Receptacle, X2 Micro Type-B Receptacle

Commit message: made changes discussed at meeting
Parts:
- moved X1 1.00 mm to (12.0, 4.00)
Connections:
- net WE1: now also X1.4, X2.5; no longer X1.2, X2.2
- net WE2: now also X1.2, X2.2; no longer X1.4, X2.5
Routing:
- net WE2: track 17.4 -> 23.1 mm
- net WE1: track 22.1 -> 18.4 mm
- net RE: track 15.7 -> 16.7 mm
- net CE: track 27.9 -> 28.9 mm
Changed lines of the file:
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@@
 <wire x1="0" y1="30" x2="0" y2="0" width="0" layer="20"/>
 <text x="7" y="19.75" size="1.27" layer="21">EmStat/MUX</text>
-<text x="5.25" y="10" size="1.016" layer="21">CE</text>
-<text x="8.5" y="10" size="1.016" layer="21">WE1</text>
-<text x="12.75" y="10" size="1.016" layer="21">RE</text>
-<text x="16.25" y="10" size="1.016" layer="21">WE2</text>
+<text x="5.25" y="9" size="1.016" layer="21">CE</text>
+<text x="8.5" y="9" size="1.016" layer="21">WE2</text>
+<text x="12.75" y="9" size="1.016" layer="21">RE</text>
+<text x="16.25" y="9" size="1.016" layer="21">WE1</text>
 </plain>
 <attributes>
@@
 </autorouter>
 <elements>
-<element name="X1" library="sensor-breakout-boards" package="TE_CONNECTIVITY_292303-1" value="Type-A Receptacle" x="12" y="5" smashed="yes">
-<attribute name="NAME" x="1" y="1" size="2" layer="25" font="vector"/>
-</element>
-<element name="X2" library="sensor-breakout-boards" package="MOLEX_0548190519" value="Micro Type-B Receptacle" x="12" y="28" smashed="yes" rot="R270">
-<attribute name="NAME" x="23" y="29" size="2" layer="25" font="vector" rot="R180"/>
-</element>
+<element name="X1" library="sensor-breakout-boards" package="TE_CONNECTIVITY_292303-1" value="Type-A Receptacle" x="12" y="4" smashed="yes"/>
+<element name="X2" library="sensor-breakout-boards" package="MOLEX_0548190519" value="Micro Type-B Receptacle" x="12" y="28" smashed="yes" rot="R270"/>
 <element name="MOUNTING1" library="sensor-breakout-boards" package="M2-MOUNTING-HOLE" value="M2-MOUNTING-HOLE" x="20" y="15"/>
 <element name="MOUNTING2" library="sensor-breakout-boards" package="M2-MOUNTING-HOLE" value="M2-MOUNTING-HOLE" x="4" y="15"/>
@@
 <wire x1="7.5" y1="24" x2="7.5" y2="15.75" width="0.6096" layer="16"/>
 <wire x1="7.5" y1="15.75" x2="8.5" y2="14.75" width="0.6096" layer="16"/>
-<wire x1="8.5" y1="14.75" x2="8.5" y2="7.71" width="0.6096" layer="16"/>
-</signal>
-<signal name="WE1">
+<wire x1="8.5" y1="14.75" x2="8.5" y2="6.71" width="0.6096" layer="16"/>
+</signal>
+<signal name="WE2">
 <contactref element="X2" pad="2"/>
 <contactref element="X1" pad="2"/>
@@
 <wire x1="9" y1="23.75" x2="9" y2="16.5" width="0.6096" layer="16"/>
 <wire x1="9" y1="16.5" x2="11" y2="14.5" width="0.6096" layer="16"/>
-<wire x1="11" y1="14.5" x2="11" y2="7.71" width="0.6096" layer="16"/>
+<wire x1="11" y1="14.5" x2="11" y2="6.71" width="0.6096" layer="16"/>
 </signal>
 <signal name="RE">
@@
 <wire x1="12" y1="22.95" x2="12" y2="18" width="0.6096" layer="16"/>
 <wire x1="12" y1="18" x2="13" y2="17" width="0.6096" layer="16"/>
-<wire x1="13" y1="17" x2="13" y2="7.71" width="0.6096" layer="16"/>
-</signal>
-<signal name="WE2">
+<wire x1="13" y1="17" x2="13" y2="6.71" width="0.6096" layer="16"/>
+</signal>
+<signal name="WE1">
 <contactref element="X2" pad="5"/>
 <contactref element="X1" pad="4"/>
 <wire x1="10.4" y1="22.95" x2="10.4" y2="17.1" width="0.6096" layer="1"/>
 <wire x1="10.4" y1="17.1" x2="15.5" y2="12" width="0.6096" layer="1"/>
-<wire x1="15.5" y1="12" x2="15.5" y2="7.71" width="0.6096" layer="1"/>
+<wire x1="15.5" y1="12" x2="15.5" y2="6.71" width="0.6096" layer="1"/>
 </signal>
 </signals>
