File: sensor-breakout-boards/wavenow-to-usb-sensor.brd (EAGLE design)
At the start: 24 x 30 mm, 4 parts, among them X1 Type-A Receptacle, X2 Micro Type-B Receptacle

Commit message: made changes discussed at meeting
Connections:
- net WE1: now also X1.4, X2.3; no longer X1.2, X2.2
- net WE2: now also X1.2, X2.2; no longer X1.4, X2.3
Routing:
- net WE2: track 17.7 -> 24.3 mm, vias 1 -> 0
- net WE1: track 24.3 -> 17.7 mm, vias 0 -> 1
Changed lines of the file:
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@@
 <text x="1" y="23.5" size="1.016" layer="21">WaveNow</text>
 <text x="5.25" y="8.5" size="1.016" layer="21">CE</text>
-<text x="8.5" y="8.5" size="1.016" layer="21">WE1</text>
+<text x="8.5" y="8.5" size="1.016" layer="21">WE2</text>
 <text x="12.5" y="8.5" size="1.016" layer="21">RE</text>
-<text x="15.5" y="8.5" size="1.016" layer="21">WE2</text>
+<text x="15.5" y="8.5" size="1.016" layer="21">WE1</text>
 </plain>
 <attributes>
@@
 </autorouter>
 <elements>
-<element name="X2" library="sensor-breakout-boards" package="MOLEX_0548190519" value="Micro Type-B Receptacle" x="12" y="28" smashed="yes" rot="R270">
-<attribute name="NAME" x="23" y="29" size="2" layer="25" font="vector" rot="R180"/>
-</element>
-<element name="X1" library="sensor-breakout-boards" package="TE_CONNECTIVITY_292303-1" value="Type-A Receptacle" x="12" y="4" smashed="yes">
-<attribute name="NAME" x="0.75" y="0.5" size="2" layer="25" font="vector"/>
-</element>
+<element name="X2" library="sensor-breakout-boards" package="MOLEX_0548190519" value="Micro Type-B Receptacle" x="12" y="28" smashed="yes" rot="R270"/>
+<element name="X1" library="sensor-breakout-boards" package="TE_CONNECTIVITY_292303-1" value="Type-A Receptacle" x="12" y="4" smashed="yes"/>
 <element name="MOUNTING1" library="sensor-breakout-boards" package="M2-MOUNTING-HOLE" value="M2-MOUNTING-HOLE" x="20" y="15"/>
 <element name="MOUNTING2" library="sensor-breakout-boards" package="M2-MOUNTING-HOLE" value="M2-MOUNTING-HOLE" x="4" y="15"/>
@@
 <wire x1="13" y1="11" x2="13" y2="6.71" width="0.6096" layer="1"/>
 </signal>
-<signal name="WE1">
+<signal name="WE2">
 <contactref element="X2" pad="2"/>
 <contactref element="X1" pad="2"/>
@@
 <wire x1="11" y1="9.25" x2="11" y2="6.71" width="0.6096" layer="16"/>
 </signal>
-<signal name="WE2">
+<signal name="WE1">
 <contactref element="X2" pad="3"/>
 <contactref element="X1" pad="4"/>
